Commit message: added spoiler part to rubot 3d model

File: src/rubot_mecanum_description/urdf/rubot_custom.urdf (robot description, URDF)
Before this commit: robot rubot, 9 links, 8 joints
Links:
- link part: geometry collision box size=0.05 0.05 0.025; visual mesh filename=package://rubot_mecanum_description/meshes/rubot/Activitat4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 scale=0.0008 0.0008 0.0008
